File: tests/kicad-project/hier_test.kicad_sch (KiCad schematic)
At the start: 1 part, among them SW301 SW_Coded

Commit message: Tests: Added test case for scaled images
Parts:
- added SW201, SW202, SW203: SW_Coded, Connector_Phoenix_MC:PhoenixContact_MCV_1,5_4-G-3.5_1x04_P3.50mm_Vertical, symbol Switch:SW_Coded
- renumbered SW301 to SW204
Other:
- note added: "AAAAA AAAAA AAAAA AAAAA AAAAA AAAAA AAAAA AAAAA"
- note added: "AAAAA AAAAA AAAAA AAAAA AAAAA AAAAA AAAAA AAAAA A"
- note added: "AAAAA AAAAA AAAAA AAAAA AAAAA AAAAA AAAAA AAAAA AA"
- note added: "AAAAA AAAAA AAAAA AAAAA AAAAA AAAAA AAAAA AAAAA AAA"
- note added: "AAAAA AAAAA AAAAA AAAAA AAAAA AAAAA AAAAA AAAAA AAAA"
- note added: "AAAAA AAAAA AAAAA AAAAA AAAAA AAAAA AAAAA AAAAA AAAAA"
- note added: "AAAAA AAAAA AAAAA AAAAA AAAAA AAAAA AAAAA AAAAA AAAAA AAAAA AAAAA AAAAA AAAAA AAAAA AAAAA AAAAA"
- note added: "AAAAA AAAAA AAAAA AAAAA AAAAA AAAAA AAAAA AAAAA AAAAA AAAAA AAAAA AAAAA AAAAA AAAAA AAAAA AAAAA A"
- note added: "AAAAA AAAAA AAAAA AAAAA AAAAA AAAAA AAAAA AAAAA AAAAA AAAAA AAAAA AAAAA AAAAA AAAAA AAAAA AAAAA AA"
- note added: "AAAAA AAAAA AAAAA AAAAA AAAAA AAAAA AAAAA AAAAA AAAAA AAAAA AAAAA AAAAA AAAAA AAAAA AAAAA AAAAA AAA"
- note added: "AAAAA AAAAA AAAAA AAAAA AAAAA AAAAA AAAAA AAAAA AAAAA AAAAA AAAAA AAAAA AAAAA AAAAA AAAAA AAAAA AAAA"
- note added: "AAAAA AAAAA AAAAA AAAAA AAAAA AAAAA AAAAA AAAAA AAAAA AAAAA AAAAA AAAAA AAAAA AAAAA AAAAA AAAAA AAAAA"
- note added: "some mirrored stuff"
- note added: "test text with "quotes""
