File: tests/kicad-project/test.kicad_sch (KiCad schematic)
At the start: 2 parts, among them SW101 SW_Coded

Commit message: Tests: Added test case for scaled images
Parts:
- added SW103, SW104: SW_Coded, Connector_Phoenix_MC:PhoenixContact_MCV_1,5_4-G-3.5_1x04_P3.50mm_Vertical, symbol Switch:SW_Coded
- gave numbers to parts that had none: 1
